File: hardware/bigdrive/ono.brd (EAGLE design)
At the start: 100 x 100 mm, 62 parts, among them Q01 IRFZ44N, Q02 IRFZ44N, Q03 IRFZ44N, Q04 IRFZ44N, Q05 IRFZ44N, Q06 IRFZ44N, Q07 IRFZ44N, Q08 IRFZ44N, Q09 IRFZ44N, Q10 IRFZ44N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

Commit message: aaaa
Parts:
- removed TLC_INS_1, TLC_INS_2: (no value), SparkFun-Connectors:1X14
- added J1, J2: (no value), SparkFun-Connectors:1X12
- TLC_OUTS_1, TLC_OUTS_2: device SparkFun-Connectors:1X14 -> SparkFun-Connectors:1X16
- moved TLC_OUTS_2 220.2 mm to (55.9, 94.0), turned to 180 degrees
- moved TLC_OUTS_1 213.8 mm to (55.9, 90.2), turned to 180 degrees
- moved CHAIN_OUT_3 201.0 mm to (64.8, 86.4)
- moved PWR_02 196.1 mm to (94.0, 90.2), turned to 180 degrees
- moved CLR_ROW_6 177.6 mm to (97.8, 54.6), turned to 270 degrees
- moved NANO_PWRS_2 174.3 mm to (54.6, 52.1), turned to 270 degrees
- moved CLR_ROW_5 172.2 mm to (94.0, 54.6), flipped to the bottom, turned to 270 degrees
- moved NANO_PWRS_1 168.9 mm to (50.8, 52.1), turned to 270 degrees
- moved CLR_ROW_4 166.8 mm to (90.2, 54.6), turned to 270 degrees
- moved CHAIN_OUT_1 166.2 mm to (64.8, 94.0)
- moved CHAIN_OUT_2 166.2 mm to (64.8, 90.2)
- moved NANO_PINS_2 159.9 mm to (21.6, 52.1), turned to 270 degrees
- moved NANO_PINS_1 158.9 mm to (25.4, 52.1), turned to 270 degrees
- moved Q17 155.1 mm to (90.2, 11.4)
- moved Q16 150.5 mm to (90.2, 17.8)
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Connections:
- removed net N$10: NANO_PWRS_1.7, NANO_PWRS_2.7, U$1.A5
- removed net N$11: NANO_PWRS_1.6, NANO_PWRS_2.6, U$1.A6
- removed net N$12: NANO_PWRS_1.5, NANO_PWRS_2.5, U$1.A7
- removed net N$15: NANO_PINS_1.4, NANO_PINS_2.4, U$1.GND1
- removed net N$17: NANO_PINS_1.11, NANO_PINS_2.11, U$1.D8
- removed net N$18: NANO_PINS_1.10, NANO_PINS_2.10, U$1.D7
- removed net N$2: NANO_PWRS_1.15, NANO_PWRS_2.15, U$1.D13
- removed net N$5: NANO_PWRS_1.12, NANO_PWRS_2.12, U$1.A0
- removed net N$6: NANO_PWRS_1.11, NANO_PWRS_2.11, U$1.A1
- removed net N$7: NANO_PWRS_1.10, NANO_PWRS_2.10, U$1.A2
- removed net N$8: NANO_PWRS_1.9, NANO_PWRS_2.9, U$1.A3
- removed net N$9: NANO_PWRS_1.8, NANO_PWRS_2.8, U$1.A4
- new net BTN_1: J1.2, J2.2, NANO_PWRS_1.12, NANO_PWRS_2.12, U$1.A0
- new net BTN_10: J1.11, J2.11, NANO_PINS_1.11, NANO_PINS_2.11, U$1.D8
- new net BTN_2: J1.3, J2.3, NANO_PWRS_1.11, NANO_PWRS_2.11, U$1.A1
- new net BTN_3: J1.4, J2.4, NANO_PWRS_1.10, NANO_PWRS_2.10, U$1.A2
- new net BTN_4: J1.5, J2.5, NANO_PWRS_1.9, NANO_PWRS_2.9, U$1.A3
- new net BTN_5: J1.6, J2.6, NANO_PWRS_1.8, NANO_PWRS_2.8, U$1.A4
- new net BTN_6: J1.7, J2.7, NANO_PWRS_1.7, NANO_PWRS_2.7, U$1.A5
- new net BTN_7: J1.8, J2.8, NANO_PWRS_1.6, NANO_PWRS_2.6, U$1.A6
- new net BTN_8: J1.9, J2.9, NANO_PWRS_1.5, NANO_PWRS_2.5, U$1.A7
- new net BTN_9: J1.10, J2.10, NANO_PINS_1.10, NANO_PINS_2.10, U$1.D7
- net 5V: now also J1.12, J2.12
- net GND: now also J1.1, J2.1, NANO_PINS_1.4, NANO_PINS_2.4, U$1.GND1
- net PWM_01: now also TLC_OUTS_1.1, TLC_OUTS_2.1
- net PWM_02: now also TLC_OUTS_1.2, TLC_OUTS_2.2
- net PWM_03: now also TLC_OUTS_1.3, TLC_OUTS_2.3
- net PWM_04: now also TLC_OUTS_1.4, TLC_OUTS_2.4
- net PWM_05: now also TLC_OUTS_1.5, TLC_OUTS_2.5
- net PWM_06: now also TLC_OUTS_1.6, TLC_OUTS_2.6
- net PWM_07: now also TLC_OUTS_1.7, TLC_OUTS_2.7
- net PWM_08: now also TLC_OUTS_1.8, TLC_OUTS_2.8
- net PWM_09: now also TLC_OUTS_1.9, TLC_OUTS_2.9
- net PWM_10: now also TLC_OUTS_1.10, TLC_OUTS_2.10
- net PWM_11: now also TLC_OUTS_1.11, TLC_OUTS_2.11
- net PWM_12: now also TLC_OUTS_1.12, TLC_OUTS_2.12
- net PWM_13: now also TLC_OUTS_1.13, TLC_OUTS_2.13
- net PWM_14: now also TLC_OUTS_1.14, TLC_OUTS_2.14
- net PWM_15: now also TLC_OUTS_1.15, TLC_OUTS_2.15
- net PWM_16: now also TLC_OUTS_1.16, TLC_OUTS_2.16
- net S_CLK: now also NANO_PWRS_1.15, NANO_PWRS_2.15, U$1.D13
Routing:
- net 5V: track 0.00 -> 30.1 mm
- net GS_CLK: track 0.00 -> 24.1 mm
- net BLANK: track 0.00 -> 24.1 mm
- net XLAT: track 0.00 -> 24.1 mm
- net PWM_16: track 0.00 -> 18.3 mm
- net S_IN: track 0.00 -> 17.8 mm
- net PWM_01: track 0.00 -> 17.0 mm
- net CLR_17: track 0.00 -> 16.5 mm
- net CLR_16: track 0.00 -> 16.1 mm
- net CLR_O4: track 0.00 -> 15.2 mm
- net CLR_O3: track 0.00 -> 15.2 mm
- net CLR_18: track 0.00 -> 15.2 mm
- net CLR_15: track 0.00 -> 15.2 mm
- net CLR_14: track 0.00 -> 15.2 mm
- net CLR_13: track 0.00 -> 15.2 mm
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- added copper zone on layer 1, net 12V
- added copper zone on layer 16, net GND
