File: hardware/bigdrive/pre.brd (EAGLE design)
At the start: 100 x 100 mm, 62 parts, among them Q01 IRFZ44N, Q02 IRFZ44N, Q03 IRFZ44N, Q04 IRFZ44N, Q05 IRFZ44N, Q06 IRFZ44N, Q07 IRFZ44N, Q08 IRFZ44N, Q09 IRFZ44N, Q10 IRFZ44N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

Commit message: aaaa
Routing:
- net XLAT: track 24.1 -> 205.3 mm, vias 0 -> 2
- net BLANK: track 33.3 -> 200.0 mm
- net GS_CLK: track 24.1 -> 190.1 mm, vias 0 -> 2
- net 5V: track 35.3 -> 189.7 mm, vias 0 -> 1
- net S_CLK: track 15.2 -> 156.0 mm
- net PWM_15: track 11.4 -> 148.1 mm
- net PWM_16: track 23.7 -> 148.6 mm, vias 0 -> 2
- net S_IN: track 16.5 -> 139.5 mm
- net CLR_O3: track 15.2 -> 135.2 mm
- net CLR_18: track 15.2 -> 132.5 mm
- net CLR_16: track 15.2 -> 127.1 mm, vias 0 -> 1
- net PWM_14: track 11.4 -> 118.5 mm, vias 0 -> 1
- net PWM_13: track 12.7 -> 117.4 mm
- net CLR_17: track 15.2 -> 113.5 mm
- net CLR_01: track 15.2 -> 106.8 mm
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- added copper zone on layer 1, net 12V
- added copper zone on layer 16, net GND
