File: hardware/bigdrive/pre.sch (EAGLE design)
At the start: 50 parts, among them Q01 IRFZ44N, Q02 IRFZ44N, Q03 IRFZ44N, Q04 IRFZ44N, Q05 IRFZ44N, Q06 IRFZ44N, Q07 IRFZ44N, Q08 IRFZ44N, Q09 IRFZ44N, Q10 IRFZ44N, Q11 IRFZ44N, Q12 IRFZ44N, Q13 IRFZ44N, Q14 IRFZ44N, Q15 IRFZ44N, Q16 IRFZ44N, Q17 IRFZ44N, Q18 IRFZ44N, U1 TLC5940NT

Commit message: aaaa
Parts:
- added CHAIN_IN_2, CHAIN_OUT_3: (no value), SparkFun-Connectors:CONN_08"
- added CLR_ROW_5, CLR_ROW_6: (no value), SparkFun-Connectors:CONN_24
- added J1, J2: (no value), SparkFun-Connectors:CONN_12
- added NANO_PINS_1, NANO_PINS_2, NANO_PWRS_1, NANO_PWRS_2: (no value), SparkFun-Connectors:CONN_15
- added TLC_OUTS_1, TLC_OUTS_2: (no value), SparkFun-Connectors:CONN_16
Connections:
- new net BTN_1: J1.2, J2.2, NANO_PWRS_1.12, NANO_PWRS_2.12, U$1.A0
- new net BTN_10: J1.11, J2.11, NANO_PINS_1.11, NANO_PINS_2.11, U$1.D8
- new net BTN_2: J1.3, J2.3, NANO_PWRS_1.11, NANO_PWRS_2.11, U$1.A1
- new net BTN_3: J1.4, J2.4, NANO_PWRS_1.10, NANO_PWRS_2.10, U$1.A2
- new net BTN_4: J1.5, J2.5, NANO_PWRS_1.9, NANO_PWRS_2.9, U$1.A3
- new net BTN_5: J1.6, J2.6, NANO_PWRS_1.8, NANO_PWRS_2.8, U$1.A4
- new net BTN_6: J1.7, J2.7, NANO_PWRS_1.7, NANO_PWRS_2.7, U$1.A5
- new net BTN_7: J1.8, J2.8, NANO_PWRS_1.6, NANO_PWRS_2.6, U$1.A6
- new net BTN_8: J1.9, J2.9, NANO_PWRS_1.5, NANO_PWRS_2.5, U$1.A7
- new net BTN_9: J1.10, J2.10, NANO_PINS_1.10, NANO_PINS_2.10, U$1.D7
- new net N$13: NANO_PWRS_1.3, NANO_PWRS_2.3, U$1.RST
- new net N$14: NANO_PINS_1.15, NANO_PINS_2.15, U$1.D12
- new net N$16: NANO_PINS_1.3, NANO_PINS_2.3, U$1.RST1
- new net N$19: NANO_PINS_1.2, NANO_PINS_2.2, U$1.RX1
- new net N$20: NANO_PINS_1.7, NANO_PINS_2.7, U$1.D4
- new net N$21: NANO_PINS_1.1, NANO_PINS_2.1, U$1.TX0
- new net N$22: NANO_PINS_1.5, NANO_PINS_2.5, U$1.D2
- new net N$3: NANO_PWRS_1.14, NANO_PWRS_2.14, U$1.3.3V
- new net N$4: NANO_PWRS_1.13, NANO_PWRS_2.13, U$1.AREF
- net 12V: now also CHAIN_IN_2.3, CHAIN_OUT_3.3, CLR_ROW_5.1, CLR_ROW_5.13, CLR_ROW_5.17, CLR_ROW_5.21, CLR_ROW_5.5, CLR_ROW_5.9, CLR_ROW_6.1, CLR_ROW_6.13, CLR_ROW_6.17, CLR_ROW_6.21, CLR_ROW_6.5, CLR_ROW_6.9, NANO_PWRS_1.1, NANO_PWRS_2.1
- net 5V: now also CHAIN_IN_2.2, CHAIN_OUT_3.2, J1.12, J2.12, NANO_PWRS_1.4, NANO_PWRS_2.4
- net BLANK: now also CHAIN_IN_2.8, CHAIN_OUT_3.8, NANO_PINS_1.13, NANO_PINS_2.13
- net CLR_01: now also CLR_ROW_5.2, CLR_ROW_6.2
- net CLR_02: now also CLR_ROW_5.3, CLR_ROW_6.3
- net CLR_05: now also CLR_ROW_5.7, CLR_ROW_6.7
- net CLR_06: now also CLR_ROW_5.8, CLR_ROW_6.8
- net CLR_07: now also CLR_ROW_5.10, CLR_ROW_6.10
- net CLR_08: now also CLR_ROW_5.11, CLR_ROW_6.11
- net CLR_09: now also CLR_ROW_5.12, CLR_ROW_6.12
- net CLR_10: now also CLR_ROW_5.14, CLR_ROW_6.14
- net CLR_11: now also CLR_ROW_5.15, CLR_ROW_6.15
- net CLR_12: now also CLR_ROW_5.16, CLR_ROW_6.16
- net CLR_13: now also CLR_ROW_5.18, CLR_ROW_6.18
- net CLR_14: now also CLR_ROW_5.19, CLR_ROW_6.19
- net CLR_15: now also CLR_ROW_5.20, CLR_ROW_6.20
- net CLR_16: now also CLR_ROW_5.22, CLR_ROW_6.22
- net CLR_17: now also CLR_ROW_5.23, CLR_ROW_6.23
- net CLR_18: now also CLR_ROW_5.24, CLR_ROW_6.24
- net CLR_O3: now also CLR_ROW_5.4, CLR_ROW_6.4
- net CLR_O4: now also CLR_ROW_5.6, CLR_ROW_6.6
- net GND: now also CHAIN_IN_2.1, CHAIN_OUT_3.1, J1.1, J2.1, NANO_PINS_1.4, NANO_PINS_2.4, NANO_PWRS_1.2, NANO_PWRS_2.2, U$1.GND2
- net GS_CLK: now also CHAIN_IN_2.6, CHAIN_OUT_3.6, NANO_PINS_1.6, NANO_PINS_2.6
- net PWM_01: now also TLC_OUTS_1.1, TLC_OUTS_2.1
- net PWM_02: now also TLC_OUTS_1.2, TLC_OUTS_2.2
- net PWM_03: now also TLC_OUTS_1.3, TLC_OUTS_2.3
- net PWM_04: now also TLC_OUTS_1.4, TLC_OUTS_2.4
- net PWM_05: now also TLC_OUTS_1.5, TLC_OUTS_2.5
- net PWM_06: now also TLC_OUTS_1.6, TLC_OUTS_2.6
- net PWM_07: now also TLC_OUTS_1.7, TLC_OUTS_2.7
- net PWM_08: now also TLC_OUTS_1.8, TLC_OUTS_2.8
- net PWM_09: now also TLC_OUTS_1.9, TLC_OUTS_2.9
- net PWM_10: now also TLC_OUTS_1.10, TLC_OUTS_2.10
- net PWM_11: now also TLC_OUTS_1.11, TLC_OUTS_2.11
- net PWM_12: now also TLC_OUTS_1.12, TLC_OUTS_2.12
- net PWM_13: now also TLC_OUTS_1.13, TLC_OUTS_2.13
- net PWM_14: now also TLC_OUTS_1.14, TLC_OUTS_2.14
- net PWM_15: now also TLC_OUTS_1.15, TLC_OUTS_2.15
- net PWM_16: now also TLC_OUTS_1.16, TLC_OUTS_2.16
- net PWM_17: now also NANO_PINS_1.8, NANO_PINS_2.8
- net PWM_18: now also NANO_PINS_1.9, NANO_PINS_2.9
- net S_CLK: now also CHAIN_IN_2.5, CHAIN_OUT_3.5, NANO_PWRS_1.15, NANO_PWRS_2.15
- net S_IN: now also CHAIN_IN_2.4, NANO_PINS_1.14, NANO_PINS_2.14
- net S_OUT: now also CHAIN_OUT_3.4
- net XLAT: now also CHAIN_IN_2.7, CHAIN_OUT_3.7, NANO_PINS_1.12, NANO_PINS_2.12
Other:
- moved on the sheet: CHAIN_IN_1, CHIAN_IN_2
